File: ice4pi.kicad_pcb (KiCad board)
At the start: 4 copper layers, 85 x 56 mm, 111 parts, among them J1 Pmod 2x6, J2 Raspberry_Pi_2_3, J3 Conn_02x12_Top_Bottom, U1 ICE40HX1K-TQ144, U2 W25Q32JVSSIQ, U3 LT3030, U4 DSC1001DI1-012.0000, U5 TFDU4101-TR3, U6 SN75160BN, U7 SN75161BN

Commit message: Release gpib4pi-1.0
Parts:
- removed C1, C16, C20, C30, C4: 10uF, Capacitor_SMD:C_0402_1005Metric
- removed C10, C11, C13, C15, C27, C29, C5, C6: 0.01uF, Capacitor_SMD:C_0402_1005Metric
- removed C12, C14, C18, C19, C2, C21, C23, C24, C25, C26, C28, C3, C32, C9: 0.1uF, Capacitor_SMD:C_0402_1005Metric
- removed C17, C22: 1 uF, Capacitor_SMD:C_0402_1005Metric
- removed C31, C8: 4.7uF, Capacitor_SMD:C_0402_1005Metric
- removed D1, D2, D3, D4, D5: LED, LED_SMD:LED_0402_1005Metric
- removed D6: CDBU0520, Diode_SMD:D_0603_1608Metric
- removed J1: Pmod 2x6, ice4pi:PinSocket_2x06_P2.54mm_Vertical_1to6_7to12
- removed R1: 1M, Resistor_SMD:R_0402_1005Metric
- removed R10, R11, R12, R13, R14: 1K, Resistor_SMD:R_0402_1005Metric
- removed R15, R16, R17, R18, R19, R2: 10K, Resistor_SMD:R_0402_1005Metric
- removed R20, R7: 100, Resistor_SMD:R_0402_1005Metric
- removed R21, R22: 47, Resistor_SMD:R_0402_1005Metric
- removed R9: 0.1, Resistor_SMD:R_0402_1005Metric
- removed U1: ICE40HX1K-TQ144, Package_QFP:TQFP-144_20x20mm_P0.5mm
- removed U2: W25Q32JVSSIQ, Package_SO:SOIC-8_3.9x4.9mm_P1.27mm
- removed U3: LT3030, ice4pi:TSSOP-20_4.4x6.5mm_P0.65mm
- removed U4: DSC1001DI1-012.0000, Oscillator:Oscillator_SMD_Abracon_ASDMB-4Pin_2.5x2.0mm
- removed U5: TFDU4101-TR3, ice4pi:TFDU4101-TR3
- removed the svg2mod at (99.3, 75.5)
Connections:
- J2 pad 10: RS232_Tx_TTL -> (no net)
- J2 pad 11: PIO0_18 -> (no net)
- J2 pad 12: PIO0_17 -> /GPIB_TE
- J2 pad 13: PIO0_16 -> (no net)
- J2 pad 15: PIO0_14 -> /GPIB_IFC
- J2 pad 16: PIO0_15 -> /GPIB_NDAC
- J2 pad 18: iCE_CREST -> /GPIB_NRFD
- J2 pad 19: iCE_MOSI -> /GPIB_DAV
- J2 pad 21: iCE_MISO -> (no net)
- J2 pad 22: iCE_CDONE -> /GPIB_ATN
- J2 pad 23: iCE_SCK -> /GPIB_SRQ
- J2 pad 24: iCE_SS_B -> /GPIB_DC
- J2 pad 26: PIO0_13 -> /GPIB_PE
- J2 pad 27: PIO0_11 -> /GPIB_REN
- J2 pad 28: PIO0_12 -> (no net)
- J2 pad 29: PIO0_10 -> /GPIB_DIO08
- J2 pad 3: PIO0_20 -> (no net)
- J2 pad 31: PIO0_08 -> /GPIB_DIO07
- J2 pad 32: PIO0_09 -> /GPIB_DIO06
- J2 pad 33: PIO0_07 -> /GPIB_DIO05
- J2 pad 35: PIO0_05 -> /GPIB_DIO04
- J2 pad 36: PIO0_06 -> /GPIB_DIO03
- J2 pad 37: PIO0_03 -> /GPIB_DIO02
- J2 pad 38: PIO0_04 -> /GPIB_DIO01
- J2 pad 40: PIO0_02 -> (no net)
- J2 pad 5: PIO0_21 -> (no net)
- J2 pad 7: PIO0_19 -> /CTRL_LED
- J2 pad 8: RS232_Rx_TTL -> (no net)
- U7 pad 14: /GPIB_EOI -> (no net)
Routing:
- net GND: track 152.7 -> 18.0 mm, vias 52 -> 17
- net +3V3: track 79.6 -> 0.00 mm, vias 23 -> 0
- net iCE_MOSI: track 67.9 -> 0.00 mm, vias 2 -> 0
- net /GPIB_DIO01: track 14.7 -> 78.9 mm, vias 0 -> 2
- net iCE_SCK: track 60.9 -> 0.00 mm, vias 3 -> 0
- net /GPIB_DIO03: track 11.1 -> 71.3 mm, vias 0 -> 2
- net /GPIB_DIO02: track 13.0 -> 72.0 mm, vias 0 -> 2
- net iCE_SS_B: track 58.3 -> 0.00 mm, vias 3 -> 0
- net iCE_MISO: track 57.9 -> 0.00 mm, vias 4 -> 0
- net /GPIB_DIO04: track 9.15 -> 64.4 mm, vias 0 -> 2
- net /GPIB_DIO06: track 6.44 -> 58.6 mm, vias 0 -> 2
- net /GPIB_DIO05: track 7.28 -> 59.3 mm, vias 0 -> 2
- net +5V: track 71.4 -> 24.5 mm, vias 24 -> 19
- net +1V2: track 46.8 -> 0.00 mm, vias 8 -> 0
- net /GPIB_DIO07: track 6.03 -> 51.7 mm, vias 0 -> 2
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- removed copper zone on In2.Cu, net +1V2
- removed copper zone on In2.Cu, net +3V3
- removed copper zone on B.Cu, net +5V
Other:
- board text added: "gpib4pi ver. 1.0"
- board text removed: "ice4pi ver. 1.2"
- board text removed: "ice4pi-gpib ver. 1.0"

Commit message: Release gpib4pi-1.1
Parts:
- R111, R112, R113, R114, R115, R116, R118, R211, R212, R213, R214, R215, R216, R218: value 3K -> 3.3K
Connections:
- J2 pad 10: (no net) -> Net-(J2-Pad10)
- J2 pad 11: (no net) -> Net-(J2-Pad11)
- J2 pad 13: (no net) -> Net-(J2-Pad13)
- J2 pad 21: (no net) -> /GPIB_EOI
- J2 pad 28: (no net) -> Net-(J2-Pad28)
- J2 pad 3: (no net) -> Net-(J2-Pad3)
- J2 pad 40: (no net) -> Net-(J2-Pad40)
- J2 pad 5: (no net) -> Net-(J2-Pad5)
- J2 pad 8: (no net) -> Net-(J2-Pad8)
- U7 pad 14: (no net) -> /GPIB_EOI
Routing:
- net /GPIB_EOI: track 0.00 -> 47.7 mm, vias 0 -> 2
Other:
- net class Default: clearance 0.2 -> 0.1
- net class Power: clearance 0.2 -> 0.1
- rule pad_to_mask_clearance: 0.051 -> 0
- rule trace_clearance: 0.2 -> 0.1
- board text added: "gpib4pi ver. 1.1"
- board text removed: "gpib4pi ver. 1.0"

Commit message: Release gpib4pi-1.2
Other:
- net class Default removed
- net class Power removed
- board text added: "gpib4pi ver. 1.2"
- board text removed: "gpib4pi ver. 1.1"

Commit message: Release gpib4pi-2.0
Parts:
- removed svg2mod: G***, ice4pi:lsi-logo-48mm
Connections:
- net +3V3 renamed +3.3V
- J2 pad 10: Net-(J2-Pad10) -> unconnected-(J2-Pad10)
- J2 pad 11: Net-(J2-Pad11) -> unconnected-(J2-Pad11)
- J2 pad 13: Net-(J2-Pad13) -> /GPIB_REN
- J2 pad 27: /GPIB_REN -> unconnected-(J2-Pad27)
- J2 pad 28: Net-(J2-Pad28) -> unconnected-(J2-Pad28)
- J2 pad 3: Net-(J2-Pad3) -> unconnected-(J2-Pad3)
- J2 pad 40: Net-(J2-Pad40) -> unconnected-(J2-Pad40)
- J2 pad 5: Net-(J2-Pad5) -> unconnected-(J2-Pad5)
- J2 pad 8: Net-(J2-Pad8) -> unconnected-(J2-Pad8)
Routing:
- net /GPIB_REN: track 32.7 -> 45.4 mm
Other:
- board text added: "gpib4pi ver. 2.0"
- board text removed: "gpib4pi ver. 1.2"

Commit message: Release gpib4pi-2.1
Parts:
- added svg2mod: G***, ice4pi:lsi-logo-48mm, F.Cu at (82.5, 103.0)
Other:
- board text added: "gpib4pi ver. 2.1"
- board text removed: "gpib4pi ver. 2.0"

Commit message: Release gpib4pi-2.2-experimental-pullup
Parts:
- added R131: 10K, Resistor_SMD:R_0402_1005Metric, F.Cu at (60.8, 80.8)
- added R132: 3.3K, Resistor_SMD:R_0402_1005Metric, F.Cu at (63.4, 80.8)
- added R133: 10K, Resistor_SMD:R_0402_1005Metric, F.Cu at (65.9, 80.8)
- added R134: 10K, Resistor_SMD:R_0402_1005Metric, F.Cu at (68.4, 80.8)
- added R135: 10K, Resistor_SMD:R_0402_1005Metric, F.Cu at (71.0, 80.8)
- added R136: 10K, Resistor_SMD:R_0402_1005Metric, F.Cu at (73.5, 80.8)
- added R137: 10K, Resistor_SMD:R_0402_1005Metric, F.Cu at (76.0, 80.8)
- added R138: 10K, Resistor_SMD:R_0402_1005Metric, F.Cu at (78.6, 80.8)
- added R231: 10K, Resistor_SMD:R_0402_1005Metric, F.Cu at (90.0, 80.8)
- added R232: 3.3K, Resistor_SMD:R_0402_1005Metric, F.Cu at (92.6, 80.8)
- added R233: 10K, Resistor_SMD:R_0402_1005Metric, F.Cu at (95.1, 80.8)
- added R234: 10K, Resistor_SMD:R_0402_1005Metric, F.Cu at (97.6, 80.8)
- added R235: 10K, Resistor_SMD:R_0402_1005Metric, F.Cu at (100.2, 80.8)
- added R236: 10K, Resistor_SMD:R_0402_1005Metric, F.Cu at (102.7, 80.8)
- added R237: 10K, Resistor_SMD:R_0402_1005Metric, F.Cu at (105.3, 80.8)
- added R238: 10K, Resistor_SMD:R_0402_1005Metric, F.Cu at (107.8, 80.8)
Routing:
- net /GPIB_SRQ: track 48.9 -> 51.9 mm
- net /GPIB_EOI: track 47.7 -> 49.0 mm
- net /GPIB_REN: track 45.4 -> 46.5 mm
- net /GPIB_NRFD: track 49.2 -> 50.3 mm
- net /GPIB_NDAC: track 49.0 -> 50.1 mm
- net /GPIB_IFC: track 45.4 -> 46.5 mm
- net /GPIB_DIO08: track 46.6 -> 47.8 mm
- net /GPIB_DIO07: track 51.7 -> 52.9 mm
- net /GPIB_DIO06: track 58.6 -> 59.7 mm
- net /GPIB_DIO05: track 59.3 -> 60.5 mm
- net /GPIB_DIO04: track 64.4 -> 65.6 mm
- net /GPIB_DIO03: track 71.3 -> 72.4 mm
- net /GPIB_DAV: track 47.9 -> 49.1 mm
- net /GPIB_ATN: track 52.2 -> 53.4 mm
- net /GPIB_DIO02: track 72.0 -> 73.2 mm
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Other:
- board text added: "gpib4pi ver. 2.2"
- board text removed: "gpib4pi ver. 2.1"
