File: ice4pi.kicad_sch (KiCad schematic)
At the start: 43 parts, among them J2 Raspberry_Pi_2_3, J3 Conn_02x12_Top_Bottom, U6 SN75160BN, U7 SN75161BN

Commit message: Release gpib4pi-2.0
Connections:
- net GPIB_REN: now also J2.13 (GPIO27); no longer J2.27 (ID_SD/GPIO0)
Other:
- title: gpib4pi-1.2 -> gpib4pi-2.0
Changed lines of the file:
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@@
   (paper "A4")
   (title_block
-    (title "gpib4pi-1.2")
+    (title "gpib4pi-2.0")
     (company "Lightside Instruments AS")
   )
@@
   (no_connect (at 185.42 45.72))
   (no_connect (at 185.42 43.18))
-  (no_connect (at 185.42 83.82))
+  (no_connect (at 226.06 43.18))
   (no_connect (at 226.06 45.72))
   (no_connect (at 185.42 66.04))
@@
     (stroke (width 0) (type default) (color 0 0 0 0))
   )
-  (wire (pts (xy 228.6 43.18) (xy 226.06 43.18))
-    (stroke (width 0) (type default) (color 0 0 0 0))
-  )
   (wire (pts (xy 81.28 111.76) (xy 81.28 101.6))
     (stroke (width 0) (type default) (color 0 0 0 0))
@@
     (stroke (width 0) (type default) (color 0 0 0 0))
   )
+  (wire (pts (xy 172.72 83.82) (xy 185.42 83.82))
+    (stroke (width 0) (type default) (color 0 0 0 0))
+  )
   (wire (pts (xy 172.72 73.66) (xy 185.42 73.66))
     (stroke (width 0) (type default) (color 0 0 0 0))
@@
     (effects (font (size 1.27 1.27)) (justify left bottom))
   )
-  (label "GPIB_REN" (at 228.6 43.18 0)
-    (effects (font (size 1.27 1.27)) (justify left bottom))
-  )
+  (label "GPIB_REN" (at 172.72 83.82 0)
+    (effects (font (size 1.27 1.27)) (justify left bottom))
+  )

Commit message: Release gpib4pi-2.1
Other:
- title: gpib4pi-2.0 -> gpib4pi-2.1
Changed lines of the file:
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@@
   (paper "A4")
   (title_block
-    (title "gpib4pi-2.0")
+    (title "gpib4pi-2.1")
     (company "Lightside Instruments AS")
   )

Commit message: Release gpib4pi-2.2-experimental-pullup
Parts:
- added R131, R133, R134, R135, R136, R137, R138, R231, R233, R234, R235, R236, R237, R238: 10K, Resistor_SMD:R_0402_1005Metric, symbol Device:R
- added R132, R232: 3.3K, Resistor_SMD:R_0402_1005Metric, symbol Device:R
Connections:
- net +3.3V: now also R131.1, R132.1, R133.1, R134.1, R135.1, R136.1, R137.1, R138.1, R231.1, R232.1, R233.1, R234.1, R235.1, R236.1, R237.1, R238.1
- net GPIB_ATN: now also R237.2
- net GPIB_DAV: now also R235.2
- net GPIB_DIO01: now also R131.2
- net GPIB_DIO02: now also R132.2
- net GPIB_DIO03: now also R133.2
- net GPIB_DIO04: now also R134.2
- net GPIB_DIO05: now also R135.2
- net GPIB_DIO06: now also R136.2
- net GPIB_DIO07: now also R137.2
- net GPIB_DIO08: now also R138.2
- net GPIB_EOI: now also R236.2
- net GPIB_IFC: now also R232.2
- net GPIB_NDAC: now also R233.2
- net GPIB_NRFD: now also R234.2
- net GPIB_REN: now also R231.2
- net GPIB_SRQ: now also R238.2
Other:
- title: gpib4pi-2.1 -> gpib4pi-2.2
